Commit message: Opus Ackerman Test
Signed-off-by: TAUverIL <TAUverIL@gmail.com>

File: src/drive_controller/urdf/cubemars_test.ros2_control.urdf.xacro (robot description, xacro)
@@ -1,4 +1,6 @@
 <?xml version="1.0"?>
 <robot name="cubemars_test" xmlns:xacro="http://www.ros.org/wiki/xacro">
+  <!-- A dummy link is required for robot_state_publisher to parse the URDF -->
+  <link name="base_link"/>
   <!-- ros2_control block using CubeMarsSystemHardware -->
   <ros2_control name="CubemarsSystem" type="system">
@@ -18,5 +20,5 @@
       <param name="enc_off">0.0</param>
       <param name="read_only">0</param>
-      <command_interface name="position"/>
+      <command_interface name="velocity"/>
       <state_interface name="position"/>
       <state_interface name="velocity"/>
@@ -32,5 +34,5 @@
       <param name="enc_off">0.0</param>
       <param name="read_only">0</param>
-      <command_interface name="position"/>
+      <command_interface name="velocity"/>
       <state_interface name="position"/>
       <state_interface name="velocity"/>
@@ -46,5 +48,5 @@
       <param name="enc_off">0.0</param>
       <param name="read_only">0</param>
-      <command_interface name="position"/>
+      <command_interface name="velocity"/>
       <state_interface name="position"/>
       <state_interface name="velocity"/>
@@ -60,5 +62,5 @@
       <param name="enc_off">0.0</param>
       <param name="read_only">0</param>
-      <command_interface name="position"/>
+      <command_interface name="velocity"/>
       <state_interface name="position"/>
       <state_interface name="velocity"/>
